File: PinSafe_hw/PinSafe/PinSafe.kicad_pcb (KiCad board)
At the start: 2 copper layers, 1 part

Commit message: hw: Add some pcb details
Parts:
- added C1: 4u7, Capacitors_SMD:C_0603_HandSoldering, F.Cu at (148.7, 64.8)
- added C10: 27p, Capacitors_SMD:C_0603_HandSoldering, F.Cu at (99.3, 99.0)
- added C11: 27p, Capacitors_SMD:C_0603_HandSoldering, F.Cu at (125.6, 94.8)
- added C12: 22p, Capacitors_SMD:C_0603_HandSoldering, F.Cu at (103.5, 99.0)
- added C13: 22p, Capacitors_SMD:C_0603_HandSoldering, F.Cu at (138.6, 66.7)
- added C14: 0.1u, Capacitors_SMD:C_0603_HandSoldering, F.Cu at (132.0, 76.4)
- added C15: 4u7, Capacitors_SMD:C_0603_HandSoldering, F.Cu at (107.6, 99.0)
- added C16: 0.1u, Capacitors_SMD:C_0603_HandSoldering, F.Cu at (153.1, 55.1)
- added C17: 0.1u, Capacitors_SMD:C_0603_HandSoldering, F.Cu at (111.8, 99.0)
- added C18: 1n, Capacitors_SMD:C_0603_HandSoldering, F.Cu at (140.3, 76.6)
- added C19: 0.1u, Capacitors_SMD:C_0603_HandSoldering, F.Cu at (147.2, 70.7)
- added C2: 4u7, Capacitors_SMD:C_0603_HandSoldering, F.Cu at (133.1, 82.3)
- added C20: 4u7, Capacitors_SMD:C_0603_HandSoldering, F.Cu at (152.9, 66.9)
- added C21: 1n, Capacitors_SMD:C_0603_HandSoldering, F.Cu at (157.6, 61.0)
- added C22: 0.1u, Capacitors_SMD:C_0603_HandSoldering, F.Cu at (115.9, 100.7)
- added C23: 0.1u, Capacitors_SMD:C_0603_HandSoldering, F.Cu at (136.2, 76.4)
- added C24: 10u, Capacitors_SMD:C_0805_HandSoldering, F.Cu at (69.8, 99.2)
- added C3: 1n, Capacitors_SMD:C_0603_HandSoldering, F.Cu at (144.6, 64.8)
- added C4: 0.1u, Capacitors_SMD:C_0603_HandSoldering, F.Cu at (74.4, 99.0)
- added C5: 1n, Capacitors_SMD:C_0603_HandSoldering, F.Cu at (82.7, 99.0)
- added C6: 0.1u, Capacitors_SMD:C_0603_HandSoldering, F.Cu at (86.9, 99.0)
- added C7: 0.1u, Capacitors_SMD:C_0603_HandSoldering, F.Cu at (91.0, 99.0)
- added C8: 0.1u, Capacitors_SMD:C_0603_HandSoldering, F.Cu at (95.2, 99.0)
- added C9: 1u, Capacitors_SMD:C_0603_HandSoldering, F.Cu at (78.6, 99.0)
- added DD1: STM32L151CCUx, Housings_DFN_QFN:QFN-48-1EP_7x7mm_Pitch0.5mm, F.Cu at (136.1, 57.9)
- added DD2: PN532, Housings_DFN_QFN:QFN-40-1EP_6x6mm_Pitch0.5mm, F.Cu at (127.3, 86.6)
- added R1: 510R, Resistors_SMD:R_0603_HandSoldering, F.Cu at (153.3, 61.0)
- added R2: 1k, Resistors_SMD:R_0603_HandSoldering, F.Cu at (157.4, 55.1)
- added R3: 2k7, Resistors_SMD:R_0603_HandSoldering, F.Cu at (142.9, 70.7)
- added XL1: CONN_3, Pin_Headers:Pin_Header_Straight_1x03, F.Cu at (126.7, 74.1)
- added XL2: ST_SWD, Pin_Headers:Pin_Header_Straight_1x04, F.Cu at (126.6, 58.3)
- added XTAL1: 8MHz, Crystals:Crystal_SMD_0603_4Pads, F.Cu at (133.2, 68.6)
- added XTAL2: CRYSTAL_H, Crystals:Crystal_SMD_0603_4Pads, F.Cu at (146.8, 57.0)
- moved SC1 58.8 mm to (123.1, 54.0)
Connections:
- SC1 pad 1: Net-(SC1-Pad1) -> /SC_VCC
- SC1 pad 10: Net-(SC1-Pad10) -> GND
- SC1 pad 2: Net-(SC1-Pad2) -> /SC_RESET
- SC1 pad 3: Net-(SC1-Pad3) -> /SC_CLK
- SC1 pad 5: Net-(SC1-Pad5) -> GND
- SC1 pad 6: Net-(SC1-Pad6) -> /SC_VPP
- SC1 pad 7: Net-(SC1-Pad7) -> /SC_IO
- SC1 pad 9: Net-(SC1-Pad9) -> /SC_STATE

Commit message: Antenna pcb add
Parts:
- added C25: 10u, Capacitors:CAP_0805, F.Cu at (132.5, 112.8)
- added C26: 0.1u, Capacitors:CAP_0603, F.Cu at (181.9, 101.8)
- added C27: 4u7, Capacitors:CAP_0603, F.Cu at (200.5, 80.5)
- added C28: 0.1u, Capacitors:CAP_0603, F.Cu at (184.4, 95.4)
- added C29: 220p, Capacitors:CAP_0603, F.Cu at (195.1, 90.1)
- added C30: 220p, Capacitors:CAP_0603, F.Cu at (170.8, 112.5)
- added C31: Cp, Capacitors:CAP_0603, F.Cu at (191.5, 90.1)
- added C32: Cp, Capacitors:CAP_0603, F.Cu at (188.0, 95.4)
- added C33: Cp, Capacitors:CAP_0603, F.Cu at (177.0, 112.4)
- added C34: Cp, Capacitors:CAP_0603, F.Cu at (191.5, 94.3)
- added D1: LED, LEDs:LED_0603, F.Cu at (149.1, 112.6)
- added D2: LED, LEDs:LED_0603, F.Cu at (145.2, 112.6)
- added DA1: TLV733xx, SOT:SOT23-5, F.Cu at (177.8, 102.9)
- added L1: 560n, Inductors:IND_0805, F.Cu at (141.2, 112.7)
- added L2: 560n, Inductors:IND_0805, F.Cu at (136.9, 112.7)
- added Q1: IRLML6302, TO_SOT_Packages_SMD:SOT-23_Handsoldering, F.Cu at (202.8, 69.4)
- added R4: R, Resistors:RES_0603, F.Cu at (200.5, 84.7)
- added R5: R, Resistors:RES_0603, F.Cu at (181.9, 106.0)
- added R6: 10k, Resistors:RES_0603, F.Cu at (207.1, 76.3)
- added R7: 0R, Resistors:RES_0603, F.Cu at (189.0, 99.6)
- added R8: 0R, Resistors:RES_0603, F.Cu at (192.6, 98.5)
- added R9: R, Resistors:RES_0603, F.Cu at (185.5, 103.8)
- added XL3: USB_MINI_B, Connectors:USBmicro_MOLEX_WM17142, F.Cu at (181.1, 71.0)
- C1, C10, C11, C12, C13, C14, C15, C16, C17, C18, C19, C2, C20, C21, C22, C23, C3, C4, C5, C6, C7, C8, C9: footprint Capacitors_SMD:C_0603_HandSoldering -> Capacitors:CAP_0603
- C24: footprint Capacitors_SMD:C_0805_HandSoldering -> Capacitors:CAP_0805
- R1, R2, R3: footprint Resistors_SMD:R_0603_HandSoldering -> Resistors:RES_0603
- XL1: footprint Pin_Headers:Pin_Header_Straight_1x03 -> Connectors:PLS-3
- XL2: footprint Pin_Headers:Pin_Header_Straight_1x04 -> Connectors:PLS-4
- XTAL1, XTAL2: footprint Crystals:Crystal_SMD_0603_4Pads -> Quartz:0503x4-4
- moved C4 133.9 mm to (207.6, 84.7)
- moved C24 129.3 mm to (196.1, 71.2)
- moved C9 123.5 mm to (200.0, 76.3)
- moved C7 118.0 mm to (207.6, 80.5)
- moved C5 116.3 mm to (198.6, 88.9)
- moved C6 115.7 mm to (202.2, 88.9)
- moved C22 91.0 mm to (203.6, 76.3)
- moved C15 81.5 mm to (189.0, 103.8)
- moved C8 69.9 mm to (163.7, 112.5)
- moved C17 65.9 mm to (177.0, 108.2)
- moved XL2 63.1 mm to (189.1, 67.2)
- moved C3 62.7 mm to (204.0, 84.7)
- moved C10 62.3 mm to (160.2, 112.5)
- moved R3 61.9 mm to (204.0, 80.5)
- moved C14 61.6 mm to (193.4, 81.7)
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Connections:
- DD1 pad 20: Net-(DD1-Pad20) -> /PN_RESET
- DD2 pad 14: Net-(DD2-Pad14) -> Net-(C12-Pad1)
- SC1 pad 1: /SC_VCC -> /SC_POWER
